Commit message: updated urdf

File: ros2_ws/src/rl12dof_urdf_description/urdf/materials.xacro (robot description, xacro)
@@ -1,4 +1,4 @@
 <?xml version="1.0" ?>
-<robot name="RL_URDF" xmlns:xacro="http://www.ros.org/wiki/xacro" >
+<robot name="rl12dof_urdf" xmlns:xacro="http://www.ros.org/wiki/xacro" >
 <material name="silver">
   <color rgba="0.700 0.700 0.700 1.000"/>

File: ros2_ws/src/rl12dof_urdf_description/urdf/rl12dof_urdf.xacro (robot description, xacro)
@@ -1,7 +1,7 @@
 <?xml version="1.0" ?>
-<robot name="RL_URDF" xmlns:xacro="http://www.ros.org/wiki/xacro">
-<xacro:include filename="$(find RL_URDF_description)/urdf/materials.xacro" />
-<xacro:include filename="$(find RL_URDF_description)/urdf/RL_URDF.ros2control" />
-<xacro:include filename="$(find RL_URDF_description)/urdf/RL_URDF.gazebo" />
+<robot name="rl12dof_urdf" xmlns:xacro="http://www.ros.org/wiki/xacro">
+<xacro:include filename="$(find rl12dof_urdf_description)/urdf/materials.xacro" />
+<xacro:include filename="$(find rl12dof_urdf_description)/urdf/rl12dof_urdf.ros2control" />
+<xacro:include filename="$(find rl12dof_urdf_description)/urdf/rl12dof_urdf.gazebo" />
 <link name="base_link">
   <inertial>
@@ -13,5 +13,5 @@
     <origin xyz="0 0 0" rpy="0 0 0"/>
     <geometry>
-      <mesh filename="file://$(find RL_URDF_description)/meshes/base_link.stl" scale="0.001 0.001 0.001"/>
+      <mesh filename="file://$(find rl12dof_urdf_description)/meshes/base_link.stl" scale="0.001 0.001 0.001"/>
     </geometry>
     <material name="silver"/>
@@ -20,5 +20,5 @@
     <origin xyz="0 0 0" rpy="0 0 0"/>
     <geometry>
-      <mesh filename="file://$(find RL_URDF_description)/meshes/base_link.stl" scale="0.001 0.001 0.001"/>
+      <mesh filename="file://$(find rl12dof_urdf_description)/meshes/base_link.stl" scale="0.001 0.001 0.001"/>
     </geometry>
   </collision>
@@ -33,5 +33,5 @@
     <origin xyz="-0.0 -0.0 -0.007807" rpy="0 0 0"/>
     <geometry>
-      <mesh filename="file://$(find RL_URDF_description)/meshes/Hip_Link_v28_1.stl" scale="0.001 0.001 0.001"/>
+      <mesh filename="file://$(find rl12dof_urdf_description)/meshes/Hip_Link_v28_1.stl" scale="0.001 0.001 0.001"/>
     </geometry>
     <material name="silver"/>
@@ -40,5 +40,5 @@
     <origin xyz="-0.0 -0.0 -0.007807" rpy="0 0 0"/>
     <geometry>
-      <mesh filename="file://$(find RL_URDF_description)/meshes/Hip_Link_v28_1.stl" scale="0.001 0.001 0.001"/>
+      <mesh filename="file://$(find rl12dof_urdf_description)/meshes/Hip_Link_v28_1.stl" scale="0.001 0.001 0.001"/>
     </geometry>
   </collision>
@@ -53,5 +53,5 @@
     <origin xyz="-0.0 -0.023241 -0.068373" rpy="0 0 0"/>
     <geometry>
-      <mesh filename="file://$(find RL_URDF_description)/meshes/Hip_Pitch_v1_1.stl" scale="0.001 0.001 0.001"/>
+      <mesh filename="file://$(find rl12dof_urdf_description)/meshes/Hip_Pitch_v1_1.stl" scale="0.001 0.001 0.001"/>
     </geometry>
     <material name="silver"/>
@@ -60,5 +60,5 @@
     <origin xyz="-0.0 -0.023241 -0.068373" rpy="0 0 0"/>
     <geometry>
-      <mesh filename="file://$(find RL_URDF_description)/meshes/Hip_Pitch_v1_1.stl" scale="0.001 0.001 0.001"/>
+      <mesh filename="file://$(find rl12dof_urdf_description)/meshes/Hip_Pitch_v1_1.stl" scale="0.001 0.001 0.001"/>
     </geometry>
   </collision>
@@ -73,5 +73,5 @@
     <origin xyz="0.0 0.002159 -0.068373" rpy="0 0 0"/>
     <geometry>
-      <mesh filename="file://$(find RL_URDF_description)/meshes/Inner_Motor_Coupling_v26_1.stl" scale="0.001 0.001 0.001"/>
+      <mesh filename="file://$(find rl12dof_urdf_description)/meshes/Inner_Motor_Coupling_v26_1.stl" scale="0.001 0.001 0.001"/>
     </geometry>
     <material name="silver"/>
@@ -80,5 +80,5 @@
     <origin xyz="0.0 0.002159 -0.068373" rpy="0 0 0"/>
     <geometry>
-      <mesh filename="file://$(find RL_URDF_description)/meshes/Inner_Motor_Coupling_v26_1.stl" scale="0.001 0.001 0.001"/>
+      <mesh filename="file://$(find rl12dof_urdf_description)/meshes/Inner_Motor_Coupling_v26_1.stl" scale="0.001 0.001 0.001"/>
     </geometry>
   </collision>
@@ -93,5 +93,5 @@
     <origin xyz="0.0 0.026289 -0.068373" rpy="0 0 0"/>
     <geometry>
-      <mesh filename="file://$(find RL_URDF_description)/meshes/Knee_Pitch_v1_1.stl" scale="0.001 0.001 0.001"/>
+      <mesh filename="file://$(find rl12dof_urdf_description)/meshes/Knee_Pitch_v1_1.stl" scale="0.001 0.001 0.001"/>
     </geometry>
     <material name="silver"/>
@@ -100,5 +100,5 @@
     <origin xyz="0.0 0.026289 -0.068373" rpy="0 0 0"/>
     <geometry>
-      <mesh filename="file://$(find RL_URDF_description)/meshes/Knee_Pitch_v1_1.stl" scale="0.001 0.001 0.001"/>
+      <mesh filename="file://$(find rl12dof_urdf_description)/meshes/Knee_Pitch_v1_1.stl" scale="0.001 0.001 0.001"/>
     </geometry>
   </collision>
@@ -113,5 +113,5 @@
     <origin xyz="0.0 0.038989 -0.068373" rpy="0 0 0"/>
     <geometry>
-      <mesh filename="file://$(find RL_URDF_description)/meshes/Outer_Motor_Coupling_v25_1.stl" scale="0.001 0.001 0.001"/>
+      <mesh filename="file://$(find rl12dof_urdf_description)/meshes/Outer_Motor_Coupling_v25_1.stl" scale="0.001 0.001 0.001"/>
     </geometry>
     <material name="silver"/>
@@ -120,5 +120,5 @@
     <origin xyz="0.0 0.038989 -0.068373" rpy="0 0 0"/>
     <geometry>
-      <mesh filename="file://$(find RL_URDF_description)/meshes/Outer_Motor_Coupling_v25_1.stl" scale="0.001 0.001 0.001"/>
+      <mesh filename="file://$(find rl12dof_urdf_description)/meshes/Outer_Motor_Coupling_v25_1.stl" scale="0.001 0.001 0.001"/>
     </geometry>
   </collision>
@@ -133,5 +133,5 @@
     <origin xyz="0.0 0.064389 -0.068373" rpy="0 0 0"/>
     <geometry>
-      <mesh filename="file://$(find RL_URDF_description)/meshes/Right_Femur_Housing_v1_1.stl" scale="0.001 0.001 0.001"/>
+      <mesh filename="file://$(find rl12dof_urdf_description)/meshes/Right_Femur_Housing_v1_1.stl" scale="0.001 0.001 0.001"/>
     </geometry>
     <material name="silver"/>
@@ -140,5 +140,5 @@
     <origin xyz="0.0 0.064389 -0.068373" rpy="0 0 0"/>
     <geometry>
-      <mesh filename="file://$(find RL_URDF_description)/meshes/Right_Femur_Housing_v1_1.stl" scale="0.001 0.001 0.001"/>
+      <mesh filename="file://$(find rl12dof_urdf_description)/meshes/Right_Femur_Housing_v1_1.stl" scale="0.001 0.001 0.001"/>
     </geometry>
   </collision>
@@ -153,5 +153,5 @@
     <origin xyz="0.0 0.086614 -0.068373" rpy="0 0 0"/>
     <geometry>
-      <mesh filename="file://$(find RL_URDF_description)/meshes/Right_Femur_Thigh_Cap_v1_1.stl" scale="0.001 0.001 0.001"/>
+      <mesh filename="file://$(find rl12dof_urdf_description)/meshes/Right_Femur_Thigh_Cap_v1_1.stl" scale="0.001 0.001 0.001"/>
     </geometry>
     <material name="silver"/>
@@ -160,5 +160,5 @@
     <origin xyz="0.0 0.086614 -0.068373" rpy="0 0 0"/>
     <geometry>
-      <mesh filename="file://$(find RL_URDF_description)/meshes/Right_Femur_Thigh_Cap_v1_1.stl" scale="0.001 0.001 0.001"/>
+      <mesh filename="file://$(find rl12dof_urdf_description)/meshes/Right_Femur_Thigh_Cap_v1_1.stl" scale="0.001 0.001 0.001"/>
     </geometry>
   </collision>
@@ -173,5 +173,5 @@
     <origin xyz="0.0 0.080962 -0.214423" rpy="0 0 0"/>
     <geometry>
-      <mesh filename="file://$(find RL_URDF_description)/meshes/Tibia_Link_v97_1.stl" scale="0.001 0.001 0.001"/>
+      <mesh filename="file://$(find rl12dof_urdf_description)/meshes/Tibia_Link_v97_1.stl" scale="0.001 0.001 0.001"/>
     </geometry>
     <material name="silver"/>
@@ -180,5 +180,5 @@
     <origin xyz="0.0 0.080962 -0.214423" rpy="0 0 0"/>
     <geometry>
-      <mesh filename="file://$(find RL_URDF_description)/meshes/Tibia_Link_v97_1.stl" scale="0.001 0.001 0.001"/>
+      <mesh filename="file://$(find rl12dof_urdf_description)/meshes/Tibia_Link_v97_1.stl" scale="0.001 0.001 0.001"/>
     </geometry>
   </collision>
@@ -193,5 +193,5 @@
     <origin xyz="0.0 0.064389 -0.068373" rpy="0 0 0"/>
     <geometry>
-      <mesh filename="file://$(find RL_URDF_description)/meshes/Knee_Drive_Gear_v22_1.stl" scale="0.001 0.001 0.001"/>
+      <mesh filename="file://$(find rl12dof_urdf_description)/meshes/Knee_Drive_Gear_v22_1.stl" scale="0.001 0.001 0.001"/>
     </geometry>
     <material name="silver"/>
@@ -200,5 +200,5 @@
     <origin xyz="0.0 0.064389 -0.068373" rpy="0 0 0"/>
     <geometry>
-      <mesh filename="file://$(find RL_URDF_description)/meshes/Knee_Drive_Gear_v22_1.stl" scale="0.001 0.001 0.001"/>
+      <mesh filename="file://$(find rl12dof_urdf_description)/meshes/Knee_Drive_Gear_v22_1.stl" scale="0.001 0.001 0.001"/>
     </geometry>
   </collision>
@@ -206,5 +206,5 @@
 <link name="Knee_Driven_Gear_v1_1">
   <inertial>
-    <origin xyz="-2.666435188826637e-16 -0.0006253228920345411 2.145816601351047e-07" rpy="0 0 0"/>
+    <origin xyz="-2.6659694766287807e-16 -0.0006253228920345411 2.145816601351047e-07" rpy="0 0 0"/>
     <mass value="0.005820129779056626"/>
     <inertia ixx="0.0" iyy="1e-06" izz="0.0" ixy="0.0" iyz="-0.0" ixz="-0.0"/>
@@ -213,5 +213,5 @@
     <origin xyz="0.0 0.080962 -0.214423" rpy="0 0 0"/>
     <geometry>
-      <mesh filename="file://$(find RL_URDF_description)/meshes/Knee_Driven_Gear_v1_1.stl" scale="0.001 0.001 0.001"/>
+      <mesh filename="file://$(find rl12dof_urdf_description)/meshes/Knee_Driven_Gear_v1_1.stl" scale="0.001 0.001 0.001"/>
     </geometry>
     <material name="silver"/>
@@ -220,5 +220,5 @@
     <origin xyz="0.0 0.080962 -0.214423" rpy="0 0 0"/>
     <geometry>
-      <mesh filename="file://$(find RL_URDF_description)/meshes/Knee_Driven_Gear_v1_1.stl" scale="0.001 0.001 0.001"/>
+      <mesh filename="file://$(find rl12dof_urdf_description)/meshes/Knee_Driven_Gear_v1_1.stl" scale="0.001 0.001 0.001"/>
     </geometry>
   </collision>
@@ -233,5 +233,5 @@
     <origin xyz="-0.003276 0.080962 -0.367069" rpy="0 0 0"/>
     <geometry>
-      <mesh filename="file://$(find RL_URDF_description)/meshes/Foot_V3_Foot_v1_1.stl" scale="0.001 0.001 0.001"/>
+      <mesh filename="file://$(find rl12dof_urdf_description)/meshes/Foot_V3_Foot_v1_1.stl" scale="0.001 0.001 0.001"/>
     </geometry>
     <material name="silver"/>
@@ -240,5 +240,5 @@
     <origin xyz="-0.003276 0.080962 -0.367069" rpy="0 0 0"/>
     <geometry>
-      <mesh filename="file://$(find RL_URDF_description)/meshes/Foot_V3_Foot_v1_1.stl" scale="0.001 0.001 0.001"/>
+      <mesh filename="file://$(find rl12dof_urdf_description)/meshes/Foot_V3_Foot_v1_1.stl" scale="0.001 0.001 0.001"/>
     </geometry>
   </collision>
